Commit message: fix error

File: robot/ur5e.urdf (robot description, URDF)
Before this commit: robot ur5e, 10 links, 9 joints
Links:
- removed link base_link
- removed link base_link_inertia
- added link base_inertia, mass 4.0; collision mesh filename=package://ur_description/meshes/ur5e/collision/base.stl; visual mesh filename=package://ur_description/meshes/ur5e/visual/base.dae
Joints:
- removed joint base_link-base_fixed_joint
- removed joint base_link-base_link_inertia
- added joint base-base_inertia: type fixed, parent base, child base_inertia, origin xyz=0 0 0 rpy=0 0 3.141592653589793
- joint shoulder_pan_joint: parent base_link_inertia -> base_inertia
- joint wrist_3-flange: origin xyz=0 0.1 0 rpy=-1.5707963267948966 0 0 -> xyz=0 0 0 rpy=0 0 0
