Commit message: add joy control & fix mobile base theta

File: robot/husky_fr3.urdf (robot description, URDF)
Before this commit: robot husky_fr3, 15 links, 14 joints
Links:
- added link v_t_link
- added link v_x_link
- added link v_y_link
Joints:
- added joint v_t_joint: type revolute, parent v_t_link, child base_link, origin xyz=0 0 -0.13228 rpy=0 0 0, axis 0 0 1, limit lower=-6.24 upper=6.24 effort=1000.0 velocity=10000.0
- added joint v_x_joint: type prismatic, parent v_x_link, child v_y_link, origin xyz=0 0 -0.13228 rpy=0 0 0, axis 1 0 0, limit lower=-10000.0 upper=-10000.0 effort=1000.0 velocity=10000.0
- added joint v_y_joint: type prismatic, parent v_y_link, child v_t_link, origin xyz=0 0 -0.13228 rpy=0 0 0, axis 0 1 0, limit lower=-10000.0 upper=-10000.0 effort=1000.0 velocity=10000.0

Commit message: update moma urdf & add srdf

File: robot/husky_fr3.urdf (robot description, URDF)
Before this commit: robot husky_fr3, 18 links, 17 joints
Links:
- added link front_left_wheel; visual mesh filename=package://mujoco_ros_sim/mujoco_menagerie/fr3_husky/assets/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
- added link front_right_wheel; visual mesh filename=package://mujoco_ros_sim/mujoco_menagerie/fr3_husky/assets/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
- added link rear_left_wheel; visual mesh filename=package://mujoco_ros_sim/mujoco_menagerie/fr3_husky/assets/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
- added link rear_right_wheel; visual mesh filename=package://mujoco_ros_sim/mujoco_menagerie/fr3_husky/assets/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
- added link top_chassis_link; visual mesh filename=package://mujoco_ros_sim/mujoco_menagerie/fr3_husky/assets/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
- added link world
- link base_link: geometry collision box size=0.7899200000000001 0.5709 0.10375; collision box size=0.9874 0.5709 0.12375
- link fr3_link0: geometry collision cylinder length=0.03 radius=0.07; collision cylinder length=0.06 radius=0.07
- link fr3_link1: geometry collision cylinder length=0.12 radius=0.065; collision cylinder length=0.2830 radius=0.07
- link fr3_link2: geometry collision cylinder length=0.12 radius=0.065; collision cylinder length=0.12 radius=0.07
- link fr3_link3: geometry collision cylinder length=0.15 radius=0.07; collision sphere radius=0.07
- link fr3_link4: geometry collision cylinder length=0.02 radius=0.07; collision cylinder length=0.02 radius=0.07
- link fr3_link5: geometry collision cylinder length=0.1 radius=0.07; collision cylinder length=0.17 radius=0.045
- link fr3_link6: geometry collision cylinder length=0.07 radius=0.07; collision cylinder length=0.08 radius=0.07
- link fr3_link7: geometry collision box size=0.071 0.071 0.041; collision cylinder length=0.05 radius=0.051
- link top_structure_link: geometry collision box size=0.38992 0.56 1.365; visual mesh filename=package://mujoco_ros_sim/mujoco_menagerie/fr3_husky/assets/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
Joints:
- added joint front_left_wheel_joint: type fixed, parent base_link, child front_left_wheel, origin xyz=0.256 0.2775 0.03282 rpy=0 0 0
- added joint front_right_wheel_joint: type fixed, parent base_link, child front_right_wheel, origin xyz=0.256 -0.2775 0.03282 rpy=0 0 0
- added joint rear_left_wheel_joint: type fixed, parent base_link, child rear_left_wheel, origin xyz=-0.256 0.2775 0.03282 rpy=0 0 0
- added joint rear_right_wheel_joint: type fixed, parent base_link, child rear_right_wheel, origin xyz=-0.256 -0.2775 0.03282 rpy=0 0 0
- added joint top_chassis_joint: type fixed, parent base_link, child top_chassis_link
- added joint world_to_vx: type fixed, parent world, child v_x_link, origin xyz=0 0 0 rpy=0 0 0
- joint base_footprint_joint: child base_footprint -> base_link; origin xyz=0 0 -0.13228 rpy=0 0 0 -> xyz=0 0 0.13228 rpy=0 0 0; parent base_link -> base_footprint
- joint v_t_joint: child base_link -> base_footprint; origin xyz=0 0 -0.13228 rpy=0 0 0 -> xyz=0 0 0 rpy=0 0 0
- joint v_x_joint: limit lower=-10000.0 upper=-10000.0 effort=1000.0 velocity=10000.0 -> lower=-10000.0 upper=10000.0 effort=1000.0 velocity=10000.0; origin xyz=0 0 -0.13228 rpy=0 0 0 -> xyz=0 0 0 rpy=0 0 0
- joint v_y_joint: limit lower=-10000.0 upper=-10000.0 effort=1000.0 velocity=10000.0 -> lower=-10000.0 upper=10000.0 effort=1000.0 velocity=10000.0; origin xyz=0 0 -0.13228 rpy=0 0 0 -> xyz=0 0 0 rpy=0 0 0

File: robot/pcv_fr3.urdf (robot description, URDF)
Before this commit: robot pcv_fr3, 21 links, 20 joints
Links:
- added link base_footprint
- added link world
- link base_link: mass 10.95 -> 107.95; geometry collision box size=0.67 0.47 0.26; visual mesh filename=package://mujoco_ros_sim/mujoco_menagerie/fr3_dyros_pcv/ass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
- link fr3_link0: geometry collision cylinder length=0.03 radius=0.07; collision cylinder length=0.06 radius=0.07
- link fr3_link1: geometry collision cylinder length=0.12 radius=0.065; collision cylinder length=0.2830 radius=0.07
- link fr3_link2: geometry collision cylinder length=0.12 radius=0.065; collision cylinder length=0.12 radius=0.07
- link fr3_link3: geometry collision cylinder length=0.15 radius=0.07; collision sphere radius=0.07
- link fr3_link4: geometry collision cylinder length=0.02 radius=0.07; collision cylinder length=0.02 radius=0.07
- link fr3_link5: geometry collision cylinder length=0.1 radius=0.07; collision cylinder length=0.17 radius=0.045
- link fr3_link6: geometry collision cylinder length=0.07 radius=0.07; collision cylinder length=0.08 radius=0.07
- link fr3_link7: geometry collision box size=0.071 0.071 0.041; collision cylinder length=0.05 radius=0.051
- link front_left_rotate: geometry collision cylinder length=0.015 radius=0.055; visual mesh filename=package://mujoco_ros_sim/mujoco_menagerie/fr3_dyros_pcv/ass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
- link front_left_steer: geometry collision cylinder length=0.03 radius=0.05; visual mesh filename=package://mujoco_ros_sim/mujoco_menagerie/fr3_dyros_pcv/ass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
- link front_right_rotate: geometry collision cylinder length=0.015 radius=0.055; visual mesh filename=package://mujoco_ros_sim/mujoco_menagerie/fr3_dyros_pcv/ass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
- link front_right_steer: geometry collision cylinder length=0.03 radius=0.05; visual mesh filename=package://mujoco_ros_sim/mujoco_menagerie/fr3_dyros_pcv/ass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
- link rear_left_rotate: geometry collision cylinder length=0.015 radius=0.055; visual mesh filename=package://mujoco_ros_sim/mujoco_menagerie/fr3_dyros_pcv/ass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
- link rear_left_steer: geometry collision cylinder length=0.03 radius=0.05; visual mesh filename=package://mujoco_ros_sim/mujoco_menagerie/fr3_dyros_pcv/ass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
- link rear_right_rotate: geometry collision cylinder length=0.015 radius=0.055; visual mesh filename=package://mujoco_ros_sim/mujoco_menagerie/fr3_dyros_pcv/ass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
- link rear_right_steer: geometry collision cylinder length=0.03 radius=0.05; visual mesh filename=package://mujoco_ros_sim/mujoco_menagerie/fr3_dyros_pcv/ass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
Joints:
- added joint base_footprint_joint: type fixed, parent base_footprint, child base_link, origin xyz=0 0 0.13228 rpy=0 0 0
- added joint world_to_vx: type fixed, parent world, child v_x_link, origin xyz=0 0 0 rpy=0 0 0
- joint v_t_joint: child base_link -> base_footprint; origin xyz=0 0 -0.13228 rpy=0 0 0 -> xyz=0 0 0 rpy=0 0 0
- joint v_x_joint: limit lower=-10000.0 upper=-10000.0 effort=1000.0 velocity=10000.0 -> lower=-10000.0 upper=10000.0 effort=1000.0 velocity=10000.0; origin xyz=0 0 -0.13228 rpy=0 0 0 -> xyz=0 0 0 rpy=0 0 0
- joint v_y_joint: limit lower=-10000.0 upper=-10000.0 effort=1000.0 velocity=10000.0 -> lower=-10000.0 upper=10000.0 effort=1000.0 velocity=10000.0; origin xyz=0 0 -0.13228 rpy=0 0 0 -> xyz=0 0 0 rpy=0 0 0

File: robot/xls_fr3.urdf (robot description, URDF)
Before this commit: robot xls_fr3, 18 links, 17 joints
Links:
- added link base_chapa; visual mesh filename=package://mujoco_ros_sim/mujoco_menagerie/fr3_xls/assets/xl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
- added link base_docking_contact
- added link base_logo_front; visual mesh filename=package://mujoco_ros_sim/mujoco_menagerie/fr3_xls/assets/xl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
- added link base_logo_left; visual mesh filename=package://mujoco_ros_sim/mujoco_menagerie/fr3_xls/assets/xl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
- added link base_logo_rear; visual mesh filename=package://mujoco_ros_sim/mujoco_menagerie/fr3_xls/assets/xl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
- added link base_logo_right; visual mesh filename=package://mujoco_ros_sim/mujoco_menagerie/fr3_xls/assets/xl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
- added link world
- link base_link: geometry collision mesh filename=package://mujoco_ros_sim/mujoco_menagerie/fr3_xls/assets/xl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; visual mesh filename=package://mujoco_ros_sim/mujoco_menagerie/fr3_xls/assets/xl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
- link fr3_link0: geometry collision cylinder length=0.03 radius=0.07; collision cylinder length=0.06 radius=0.07
- link fr3_link1: geometry collision cylinder length=0.12 radius=0.065; collision cylinder length=0.2830 radius=0.07
- link fr3_link2: geometry collision cylinder length=0.12 radius=0.065; collision cylinder length=0.12 radius=0.07
- link fr3_link3: geometry collision cylinder length=0.15 radius=0.07; collision sphere radius=0.07
- link fr3_link4: geometry collision cylinder length=0.02 radius=0.07; collision cylinder length=0.02 radius=0.07
- link fr3_link5: geometry collision cylinder length=0.1 radius=0.07; collision cylinder length=0.17 radius=0.045
- link fr3_link6: geometry collision cylinder length=0.07 radius=0.07; collision cylinder length=0.08 radius=0.07
- link fr3_link7: geometry collision box size=0.071 0.071 0.041; collision cylinder length=0.05 radius=0.051
- link front_left_wheel_link: geometry collision cylinder length=0.087 radius=0.127; visual mesh filename=package://mujoco_ros_sim/mujoco_menagerie/fr3_xls/assets/xl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
- link front_right_wheel_link: geometry collision cylinder length=0.087 radius=0.127; visual mesh filename=package://mujoco_ros_sim/mujoco_menagerie/fr3_xls/assets/xl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
- link rear_left_wheel_link: geometry collision cylinder length=0.087 radius=0.127; visual mesh filename=package://mujoco_ros_sim/mujoco_menagerie/fr3_xls/assets/xl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
- link rear_right_wheel_link: geometry collision cylinder length=0.087 radius=0.127; visual mesh filename=package://mujoco_ros_sim/mujoco_menagerie/fr3_xls/assets/xl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
Joints:
- added joint base_docking_joint: type fixed, parent base_link, child base_docking_contact, origin xyz=0.35 0 0.09 rpy=0 0 0
- added joint base_logo_front_joint: type fixed, parent base_link, child base_logo_front, origin xyz=0.345 0.0 0.0 rpy=0 0 -1.5707963267948966
- added joint base_logo_left_joint: type fixed, parent base_link, child base_logo_left, origin xyz=0.0 0.28931 0.29062 rpy=0 0 0
- added joint base_logo_rear_joint: type fixed, parent base_link, child base_logo_rear, origin xyz=-0.345 0.0 0.0 rpy=0 0 1.5707963267948966
- added joint base_logo_right_joint: type fixed, parent base_link, child base_logo_right, origin xyz=0.0 -0.28931 0.29062 rpy=0 0 3.141592653589793
- added joint base_tapa_joint: type fixed, parent base_link, child base_chapa, origin xyz=0.0 0 0.38062 rpy=0 0 0
- added joint world_to_vx: type fixed, parent world, child v_x_link, origin xyz=0 0 0 rpy=0 0 0
- joint base_footprint_joint: child base_footprint -> base_link; origin xyz=0 0 -0.127 rpy=0 0 0 -> xyz=0 0 0.127 rpy=0 0 0; parent base_link -> base_footprint
- joint v_t_joint: child base_link -> base_footprint; origin xyz=0 0 -0.13228 rpy=0 0 0 -> xyz=0 0 0 rpy=0 0 0
- joint v_x_joint: limit lower=-10000.0 upper=-10000.0 effort=1000.0 velocity=10000.0 -> lower=-10000.0 upper=10000.0 effort=1000.0 velocity=10000.0; origin xyz=0 0 -0.13228 rpy=0 0 0 -> xyz=0 0 0 rpy=0 0 0
- joint v_y_joint: limit lower=-10000.0 upper=-10000.0 effort=1000.0 velocity=10000.0 -> lower=-10000.0 upper=10000.0 effort=1000.0 velocity=10000.0; origin xyz=0 0 -0.13228 rpy=0 0 0 -> xyz=0 0 0 rpy=0 0 0
